File: Schematics/master_board/master_board.kicad_sch (KiCad schematic)
At the start: 31 parts, among them J1 Conn_01x01_Male, SW1 SW_Push, SW2 SW_Push, U1 NCP1117-3.3_SOT223, U2 RP2040, U3 W25Q64JVXGIQ, Y1 Crystal_GND2

Commit message: Update master schematics
Parts:
- removed C13: 100nF, symbol Device:C
- removed J1: Conn_01x01_Male, symbol Connector:Conn_01x01_Male
- removed R6: 10k, symbol Device:R
- removed SWD1: Conn_01x03_Female, symbol Connector:Conn_01x03_Female
- removed U3: W25Q64JVXGIQ, symbol Flash_Memory:W25Q64JVXGIQ
- removed USB1: USB_C_Receptacle, symbol Connector:USB_C_Receptacle
- removed Y1: Crystal_GND2, symbol Device:Crystal_GND2
- added C? (x2): 100n, symbol Device:C
- added D?: LED_RGB_EP, symbol Device:LED_RGB_EP
- added J?: 2x5x1.27mm, symbol Connector_Generic:Conn_02x05_Odd_Even
- added J?: USB_C_Receptacle_USB2.0, symbol Connector:USB_C_Receptacle_USB2.0
- added R? (x3): 49R9, symbol Device:R
- added R? (x2): 27R4, symbol Device:R
- added R? (x3): 1k, symbol Device:R
- added R? (x2): 10k, symbol Device:R
- added SW?: SW_Push, symbol Switch:SW_Push
- added U?: W25Q16JVSSIQ, symbol Merrick_Symbols_KiCad6:W25Q16JVSSIQ
- added Y?: ABLS-12.000MHZ-B4-T, symbol Device:Crystal
- C1, C2: value 1uF -> 10u
- C3, C4: value 10pF -> 27p
- R4, R5: value R -> 10k
Connections:
- net +3V3: now also C2.2, C?.1, C?.1, D?.4 (BA), D?.5 (GA), D?.6 (RA), J?.1 (Pin_1), R?.2, U?.8 (VCC); no longer C2.1
- net GND: now also C2.1, C?.2, C?.2, J?.3 (Pin_3), J?.5 (Pin_5), J?.9 (Pin_9), J?.A1 (GND), J?.A12 (GND), J?.B1 (GND), J?.B12 (GND), J?.S1 (SHIELD), SW?.2, U?.4 (GND); no longer C2.2
- net GPIO17: no longer R4.2, R5.2, SW1.1, SW2.1
- net GPIO2: now also R?.1
- net GPIO3: now also R?.1
- net GPIO4: now also R?.1
- net QSPI_NSS: now also R?.1, R?.2, U?.1 (~{CS})
- net QSPI_SCLK: now also U?.6 (CLK)
- net QSPI_SD0: now also U?.5 (DI(IO0))
- net QSPI_SD1: now also U?.2 (DO(IO1))
- net QSPI_SD2: now also U?.3 (IO2)
- net QSPI_SD3: now also U?.7 (IO3)
- net SWCLK: now also R?.2
- net SWDIO: now also R?.2
- net XTAL_IN: now also Y?.2
- net at R1.1: now also J?.A5 (CC1)
- net at R2.1: now also J?.B5 (CC2)
- net USB_D-I: now reaches U2.46 (USB_DM)
- net USB_D-I: now also R?.2
- net USB_D+I: now reaches U2.47 (USB_DP)
- net USB_D+I: now also R?.2
- net at C4.2, R3.1: now also Y?.1
- net +5V renamed VBUS
- net VBUS: now also J?.A4 (VBUS), J?.A9 (VBUS), J?.B4 (VBUS), J?.B9 (VBUS)
- net RESET_N renamed RUN_N
- net RUN_N: now also R5.2, SW2.1, R?.2
- net SPI0_RX renamed GPIO16
- net SPI0_SCLK renamed GPIO18
- net SPI0_TX renamed GPIO19
- new net: J?.10 (Pin_10), R?.1
- new net: J?.2 (Pin_2), R?.1
- new net: J?.4 (Pin_4), R?.1
- new net BOOTSEL_N: R?.1, SW?.1
- new net LB: D?.3 (BK), R?.2
- new net LG: D?.2 (GK), R?.2
- new net LR: D?.1 (RK), R?.2
- new net RESCAN_N: R4.2, SW1.1
- new net USB_D+: J?.A6 (D+), J?.B6 (D+), R?.1
- new net USB_D-: J?.A7 (D-), J?.B7 (D-), R?.1
- no-connect marks 12 -> 6
Other:
- added sheet 5-to-32 (5-to-32.kicad_sch)
- note added: "1ks sufficient (use PWM)"
- note added: "1uF caps MUST be close to pin44/45, use 0402 ceramics"
- note added: "BOOTSEL"
- note added: "CRYSTAL OSCILLATOR"
- note added: "Closing switch will pull flash CSN to GND."
- note added: "Connect ALL DVDD/IOVDD pins in routing to decoupling caps"
- note added: "I(max)=500mA"
- note added: "LDO REGULATOR"
- note added: "MASTER BOARD"
- note added: "MCU + DECOUPLING CAPS"
- note added: "NETS"
- note added: "No ESD protection (TVS diodes)"
- note added: "No ESD protection No common-mode choke"
- note added: "RESCAN"
- note added: "RESET"
- note added: "RGB LED"
- note added: "SWD HEADER"
- note added: "SWD available for dbg/prog"
- note added: "USB Termination resistors should be placed near chip"
- note added: "USB-C HEADER"
- note removed: "1uF must be close to pin44, use 0402 ceramics"
- note removed: "1uF must be close to pin45, use 0402 ceramics"
- note removed: "Connect ALL DVDD pins in routing to decoupling caps"
- note removed: "Connect ALL IOVDD pins in routing to decoupling caps"
- note removed: "Crystal Oscillator"
- note removed: "LDO"
- note removed: "MCU + Decoupling Caps"
- note removed: "Rescan Button"
- note removed: "Reset Button"
- note removed: "SWD Connections / Debug"
- note removed: "SWD available for programming"
- note removed: "USB is N/C on module boards"
- note removed: "USB-C"
- moved on the sheet: C1, C10, C11, C12, C14, C15, C16, C2, C3, C4, C5, C6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

Commit message: Add haptic feedback to master board
Parts:
- added R16, R17: 1k, symbol Device:R
- added U4, U5: 316040001, symbol merricks_lib:316040001
- gave numbers to parts that had none: 18
- renumbered C11 to C10, C12 to C11, C3 to C12, C4 to C13, C5 to C4, C6 to C5, C7 to C6, C8 to C7, C9 to C8, C10 to C9, R5 to R12, R3 to R14, R1 to R7, R2 to R8, R4 to R9
Connections:
- net GND: now also U4.2 (GND), U5.2 (GND)
- net GPIO5: now also R16.1
- net GPIO6: now also R17.1
- net GPIO10 renamed A2
- net GPIO11 renamed A1
- net GPIO12 renamed A0
- net GPIO16 renamed SPI0_RX
- net GPIO18 renamed SPI0_SCLK
- net GPIO19 renamed SPI0_TX
- net GPIO7 renamed E0N_B
- net GPIO8 renamed E0N_A
- net GPIO9 renamed A3
- new net: R17.2, U5.1 (VCC)
- new net: R16.2, U4.1 (VCC)
Other:
- note added: "HAPTIC FEEDBACK"
- note added: "MODULE DECODER"
- moved on the sheet: C12, C13, R14, Y1

Commit message: Assigned master board footprints
Parts:
- C1, C10, C11, C12, C13, C14, C15, C16, C17, C2, C3, C4, C5, C6, C7, C8, C9: footprint (none) -> Capacitor_SMD:C_0402_1005Metric
- J1: footprint (none) -> Connector_PinHeader_1.27mm:PinHeader_2x05_P1.27mm_Vertical
- J2: footprint (none) -> Connector_USB:USB_C_Plug_Molex_105444
- R1, R10, R11, R12, R13, R14, R15, R16, R17, R2, R3, R4, R5, R6, R7, R8, R9: footprint (none) -> Resistor_SMD:R_01005_0402Metric
- U3: footprint (none) -> W25Q16JVSSIQ:SOIC127P790X216-8N
- Y1: footprint (none) -> ABLS-12:XTAL_ABLS-12.000MHZ-B4-T
