File: Schematics/master_board/5-to-32.kicad_sch (KiCad schematic)
At the start: 3 parts

Commit message: Footprint integration
Parts:
- gave numbers to parts that had none: 3
Connections:
- net A0_B is gone; now on net A0: U7.23 (A0)
- net A1_B is gone; now on net A1: U7.22 (A1)
- net A2_B is gone; now on net A2: U7.21 (A2)
- net A3_B is gone; now on net A3: U7.20 (A3)
- net E1N_A is gone; now on net GND: U6.19 (E1N)
- net E1N_B is gone; now on net GND: U7.19 (E1N)
- net A0_A renamed A0
- net A1_A renamed A1
- net A2_A renamed A2
- net A3_A renamed A3
