File: Schematics/module_components/module_components.kicad_sch (KiCad schematic)
At the start: 16 parts

Commit message: Added footprints to resistors, capcacitors, potentiometers, etc.
Parts:
- added C1: C, Capacitor_SMD:C_0402_1005Metric, symbol Device:C
- added D1: LED_ARGB, symbol Device:LED_ARGB
- added R3, R4, R5: R, Resistor_SMD:R_0402_1005Metric, symbol Device:R
- added RV2: R_Potentiometer, Potentiometer_SMD:Potentiometer_ACP_CA6-VSMD_Vertical, symbol Device:R_Potentiometer
- R1, R2, R6, R7, R8, R9: renamed from R?; footprint (none) -> Resistor_SMD:R_0402_1005Metric
- RV1: renamed from RV?; footprint (none) -> Potentiometer_THT:Potentiometer_Bourns_PTA3043_Single_Slide
- SW1, SW3, SW4, SW5, SW6: renamed from SW?; footprint (none) -> Button_Switch_THT:Push_E-Switch_KS01Q01
- gave numbers to parts that had none: 4
Connections:
- net +3.3V: now also C1.1, D1.1 (A), RV2.1
- net GND: now also C1.2, RV2.3
- net SLIDE: now also RV2.2
- new net BLUE: D1.4 (BK), R5.2
- new net GREEN: D1.3 (GK), R4.2
- new net LED_B: R5.1
- new net LED_G: R4.1
- new net LED_R: R3.1
- new net RED: D1.2 (RK), R3.2
Other:
- note added: "LED Component"
- note added: "Twist Switch Component"
- moved on the sheet: R2, SW1
