File: schematics/master_board/5-to-32.kicad_sch (KiCad schematic)
At the start: 22 parts, among them M1 Conn_01x06_Male, M10 Conn_01x06_Male, M11 Conn_01x06_Male, M12 Conn_01x06_Male, M13 Conn_01x06_Male, M14 Conn_01x06_Male, M15 Conn_01x06_Male, M16 Conn_01x06_Male, M17 Conn_01x06_Male, M18 Conn_01x06_Male, M19 Conn_01x06_Male, M2 Conn_01x06_Male, M20 Conn_01x06_Male, M3 Conn_01x06_Male, M4 Conn_01x06_Male, M5 Conn_01x06_Male, M6 Conn_01x06_Male, M7 Conn_01x06_Male, M8 Conn_01x06_Male, M9 Conn_01x06_Male, U4 74HCT154PW,118, U5 74HCT154PW,118

Commit message: initial master board rev b
Parts:
- added TP10, TP11, TP12, TP13, TP4, TP5, TP6, TP7, TP8, TP9: TestPoint, TestPoint:TestPoint_Pad_D4.0mm, symbol Connector:TestPoint
Connections:
- net +3V3: now also TP4.1
- net GND: now also TP5.1
- net SPI0_RX: now also TP6.1
- net SPI0_SCLK: now also TP7.1
- net SPI0_TX: now also TP8.1
- net SPI_CSN11: now also TP11.1
- net SPI_CSN15: now also TP12.1
- net SPI_CSN19: now also TP13.1
- net SPI_CSN3: now also TP9.1
- net SPI_CSN7: now also TP10.1
- net SPI_CSN20: no longer names the net of U5.5 (Y4N)
- net SPI_CSN21: no longer names the net of U5.6 (Y5N)
- net SPI_CSN22: no longer names the net of U5.7 (Y6N)
- net SPI_CSN23: no longer names the net of U5.8 (Y7N)
- net SPI_CSN24: no longer names the net of U5.9 (Y8N)
- net SPI_CSN25: no longer names the net of U5.10 (Y9N)
- net SPI_CSN26: no longer names the net of U5.11 (Y10N)
- net SPI_CSN27: no longer names the net of U5.13 (Y11N)
- net SPI_CSN28: no longer names the net of U5.14 (Y12N)
- net SPI_CSN29: no longer names the net of U5.15 (Y13N)
- net SPI_CSN30: no longer names the net of U5.16 (Y14N)
- net SPI_CSN31: no longer names the net of U5.17 (Y15N)
Other:
- note added: "TEST POINTS"

Commit message: square test points, fix up routing
Parts:
- TP10, TP11, TP12, TP13, TP4, TP5, TP6, TP7, TP8, TP9: footprint TestPoint:TestPoint_Pad_D4.0mm -> TestPoint:TestPoint_Pad_2.5x2.5mm
- renumbered M1 to M0, M2 to M1, M11 to M10, M12 to M11, M13 to M12, M14 to M13, M15 to M14, M16 to M15, M17 to M16, M18 to M17, M19 to M18, M20 to M19, M3 to M2, M4 to M3, M5 to M4, M6 to M5, M7 to M6, M8 to M7, M9 to M8, M10 to M9
