File: schematics/master_board/master_board.kicad_pcb (KiCad board)
At the start: 2 copper layers, 156 x 156 mm, 71 parts, among them J1 USB_C_Receptacle_USB2.0, J2 Conn_01x04_Male, J3 Conn_01x04_Female, M1 Conn_01x06_Male, M10 Conn_01x06_Male, M11 Conn_01x06_Male, M12 Conn_01x06_Male, M13 Conn_01x06_Male, M14 Conn_01x06_Male, M15 Conn_01x06_Male, M16 Conn_01x06_Male, M17 Conn_01x06_Male, M18 Conn_01x06_Male, M19 Conn_01x06_Male, M2 Conn_01x06_Male, M20 Conn_01x06_Male, M3 Conn_01x06_Male, M4 Conn_01x06_Male, M5 Conn_01x06_Male, M6 Conn_01x06_Male, M7 Conn_01x06_Male, M8 Conn_01x06_Male, M9 Conn_01x06_Male, SW1 SW_Push, SW2 SW_Push, SW3 SW_Push, U1 NCP1117-3.3_SOT223, U2 RP2040, U3 W25Q16JVSSIQ, U4 74HCT154PW,118, U5 74HCT154PW,118, Y1 ABLS-12.000MHZ-B4-T

Commit message: initial master board rev b
Parts:
- removed the J2 at (155.6, 23.4)
- removed the R6 at (150.0, 29.2)
- added J1: Conn_01x03_MountingPin, Connector_JST:JST_SH_BM03B-SRSS-TB_1x03-1MP_P1.00mm_Vertical, F.Cu at (151.9, 22.5)
- added TP1: TestPoint, TestPoint:TestPoint_Pad_2.5x2.5mm, F.Cu at (159.3, 22.5)
- added TP10: TestPoint, TestPoint:TestPoint_Pad_D4.0mm, F.Cu at (66.8, 160.0)
- added TP11: TestPoint, TestPoint:TestPoint_Pad_D4.0mm, F.Cu at (98.3, 160.0)
- added TP12: TestPoint, TestPoint:TestPoint_Pad_D4.0mm, F.Cu at (129.8, 160.0)
- added TP13: TestPoint, TestPoint:TestPoint_Pad_D4.0mm, F.Cu at (161.3, 160.0)
- added TP2: TestPoint, TestPoint:TestPoint_Pad_2.5x2.5mm, F.Cu at (139.4, 22.5)
- added TP3: TestPoint, TestPoint:TestPoint_Pad_2.5x2.5mm, F.Cu at (29.1, 22.5)
- added TP4: TestPoint, TestPoint:TestPoint_Pad_D4.0mm, F.Cu at (84.5, 167.0)
- added TP5: TestPoint, TestPoint:TestPoint_Pad_D4.0mm, F.Cu at (89.8, 167.0)
- added TP6: TestPoint, TestPoint:TestPoint_Pad_D4.0mm, F.Cu at (95.0, 167.0)
- added TP7: TestPoint, TestPoint:TestPoint_Pad_D4.0mm, F.Cu at (100.2, 167.0)
- added TP8: TestPoint, TestPoint:TestPoint_Pad_D4.0mm, F.Cu at (105.5, 167.0)
- added TP9: TestPoint, TestPoint:TestPoint_Pad_D4.0mm, F.Cu at (35.3, 160.0)
- J3: value Conn_01x04_Female -> Conn_01x04_Male
- R11: renamed from R12; value 1k -> 10k
- R14: renamed from R15; value DNF -> 10k
- R15: renamed from R16; value 1k -> 49R9
- R16: renamed from R17; value 1k -> 49R9
- R8: renamed from R9; value 1k -> 10k
- moved J3 7.65 mm to (46.5, 22.5), turned to -90 degrees
- moved R5 3.07 mm to (150.9, 27.6)
- moved R8 2.94 mm to (154.3, 33.0), turned to 0 degrees
- moved R4 2.68 mm to (152.9, 27.6)
- moved R15 1.10 mm to (38.9, 25.6)
- moved R16 1.10 mm to (46.5, 25.6)
- renumbered J1 to J2, R11 to R10, R13 to R12, R14 to R13, R7 to R6, R8 to R7, R10 to R9
Connections:
- J3 pad 1: /CONN_HAP_L -> /CONN_HAP_R
- J3 pad 4: /CONN_HAP_R -> /CONN_HAP_L
- U2 pad 16: /GPIO13 -> unconnected-(U2-Pad16)
- U2 pad 17: /GPIO14 -> unconnected-(U2-Pad17)
- U2 pad 18: /GPIO15 -> unconnected-(U2-Pad18)
- U2 pad 2: /GPIO0 -> unconnected-(U2-Pad2)
- U2 pad 3: /GPIO1 -> unconnected-(U2-Pad3)
- U2 pad 31: /GPIO20 -> unconnected-(U2-Pad31)
- U2 pad 32: /GPIO21 -> unconnected-(U2-Pad32)
- U2 pad 34: /GPIO22 -> unconnected-(U2-Pad34)
- U2 pad 35: /GPIO23 -> unconnected-(U2-Pad35)
- U2 pad 36: /GPIO24 -> unconnected-(U2-Pad36)
- U2 pad 37: /GPIO25 -> unconnected-(U2-Pad37)
- U2 pad 38: /GPIO26_ADC0 -> unconnected-(U2-Pad38)
- U2 pad 39: /GPIO27_ADC1 -> unconnected-(U2-Pad39)
- U2 pad 40: /GPIO28_ADC2 -> unconnected-(U2-Pad40)
- U2 pad 41: /GPIO29_ADC3 -> unconnected-(U2-Pad41)
- U5 pad 10: /5-to-32/SPI_CSN25 -> unconnected-(U5-Pad10)
- U5 pad 11: /5-to-32/SPI_CSN26 -> unconnected-(U5-Pad11)
- U5 pad 13: /5-to-32/SPI_CSN27 -> unconnected-(U5-Pad13)
- U5 pad 14: /5-to-32/SPI_CSN28 -> unconnected-(U5-Pad14)
- U5 pad 15: /5-to-32/SPI_CSN29 -> unconnected-(U5-Pad15)
- U5 pad 16: /5-to-32/SPI_CSN30 -> unconnected-(U5-Pad16)
- U5 pad 17: /5-to-32/SPI_CSN31 -> unconnected-(U5-Pad17)
- U5 pad 5: /5-to-32/SPI_CSN20 -> unconnected-(U5-Pad5)
- U5 pad 6: /5-to-32/SPI_CSN21 -> unconnected-(U5-Pad6)
- U5 pad 7: /5-to-32/SPI_CSN22 -> unconnected-(U5-Pad7)
- U5 pad 8: /5-to-32/SPI_CSN23 -> unconnected-(U5-Pad8)
- U5 pad 9: /5-to-32/SPI_CSN24 -> unconnected-(U5-Pad9)
Routing:
- net SPI0_SCLK: track 646.3 -> 668.2 mm
- net SPI0_TX: track 647.6 -> 668.7 mm
- net SPI0_RX: track 645.8 -> 665.2 mm
- net +3V3: track 875.2 -> 892.1 mm
- net GND: track 110.8 -> 123.3 mm
- net /RESCAN_N: track 78.5 -> 87.9 mm
- net /5-to-32/SPI_CSN7: track 148.8 -> 158.0 mm
- net /5-to-32/SPI_CSN19: track 224.0 -> 233.2 mm
- net /5-to-32/SPI_CSN15: track 199.3 -> 208.5 mm
- net /5-to-32/SPI_CSN11: track 164.6 -> 173.9 mm
- net /5-to-32/SPI_CSN3: track 126.6 -> 134.9 mm
- net /CONN_RUN_N: track 5.85 -> 0.00 mm
- net unconnected-(J1-PadMP): track 0.00 -> 4.60 mm
- net /CONN_SWDIO: track 6.33 -> 3.27 mm
- net /BOOTSEL_N: track 44.8 -> 47.7 mm
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
Commit message: square test points, fix up routing
Parts:
- TP10, TP11, TP12, TP13, TP4, TP5, TP6, TP7, TP8, TP9: footprint TestPoint:TestPoint_Pad_D4.0mm -> TestPoint:TestPoint_Pad_2.5x2.5mm
- moved U4 9.21 mm to (58.0, 38.0), turned to 90 degrees
- moved U5 4.80 mm to (77.3, 38.0), turned to 90 degrees
- moved R7 0.38 mm to (117.8, 27.8)
- renumbered M1 to M0, M2 to M1, M11 to M10, M12 to M11, M13 to M12, M14 to M13, M15 to M14, M16 to M15, M17 to M16, M18 to M17, M19 to M18, M20 to M19, M3 to M2, M4 to M3, M5 to M4, M6 to M5, M7 to M6, M8 to M7, M9 to M8, M10 to M9
Routing:
- net /5-to-32/SPI_CSN4: track 56.5 -> 32.6 mm
- net /5-to-32/SPI_CSN5: track 87.2 -> 64.2 mm
- net /5-to-32/SPI_CSN6: track 118.0 -> 95.8 mm
- net /5-to-32/SPI_CSN7: track 158.0 -> 136.7 mm
- net /5-to-32/SPI_CSN8: track 82.7 -> 62.1 mm
- net /5-to-32/SPI_CSN9: track 113.4 -> 93.7 mm
- net /5-to-32/SPI_CSN10: track 144.2 -> 125.2 mm
- net /5-to-32/SPI_CSN16: track 128.5 -> 112.5 mm
- net /5-to-32/SPI_CSN17: track 160.5 -> 145.2 mm
- net /5-to-32/SPI_CSN18: track 192.1 -> 177.4 mm
- net /5-to-32/SPI_CSN19: track 233.2 -> 219.2 mm
- net A3: track 48.7 -> 40.2 mm, vias 3 -> 2
- net E0N_A: track 43.1 -> 35.5 mm
- net A2: track 49.2 -> 41.9 mm, vias 3 -> 2
- net A1: track 49.8 -> 43.7 mm, vias 3 -> 2
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Other:
- board text added: "Made with <3: Yu-yang Hsieh, Britton McLeavy, Caleb O'Malley, Evan Zhang, Merrick Ryman"
- board text added: "Revision Date: 03/03/2023"

Commit message: add gerbers
Changed lines of the file:
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@@
       (psnegative false)
       (psa4output false)
-      (plotreference false)
+      (plotreference true)
       (plotvalue false)
       (plotinvisibletext false)
@@
     (pad "3" smd roundrect (at 1 1.325) (size 0.6 1.55) (layers "F.Cu" "F.Paste" "F.Mask") (roundrect_rratio 0.25)
       (net 10 "/CONN_SWDIO") (pinfunction "Pin_3") (pintype "passive"))
-    (pad "MP" smd roundrect (at -2.3 -1.2) (size 1.2 1.8) (layers "F.Cu" "F.Paste" "F.Mask") (roundrect_rratio 0.208333)
+    (pad "MP" smd roundrect (at -2.3 -1.2) (size 1.2 1.8) (layers "F.Cu" "F.Paste" "F.Mask") (roundrect_rratio 0.2083333333)
       (net 93 "unconnected-(J1-PadMP)") (pinfunction "MountPin") (pintype "passive+no_connect"))
-    (pad "MP" smd roundrect (at 2.3 -1.2) (size 1.2 1.8) (layers "F.Cu" "F.Paste" "F.Mask") (roundrect_rratio 0.208333)
+    (pad "MP" smd roundrect (at 2.3 -1.2) (size 1.2 1.8) (layers "F.Cu" "F.Paste" "F.Mask") (roundrect_rratio 0.2083333333)
       (net 93 "unconnected-(J1-PadMP)") (pinfunction "MountPin") (pintype "passive+no_connect"))
     (model "${KICAD6_3DMODEL_DIR}/Connector_JST.3dshapes/JST_GH_BM03B-GHS-TBT_1x03-1MP_P1.25mm_Vertical.step"
@@
     (effects (font (size 1 1) (thickness 0.2)) (justify mirror))
   )
-  (gr_text "PROTOTROLLER" (at 45 30.66) (layer "F.SilkS")
+  (gr_text "PROTOTROLLER" (at 45.01 31.05) (layer "F.SilkS")
     (effects (font (size 1.5 1.5) (thickness 0.3) italic))
   )
@@
     (effects (font (size 1 1) (thickness 0.2)))
   )
-  (gr_text "USB" (at 126.2 21.4 90) (layer "F.SilkS")
+  (gr_text "USB" (at 126.2 22.5 90) (layer "F.SilkS")
     (effects (font (size 1 1) (thickness 0.2)))
   )
@@
     (effects (font (size 1 1) (thickness 0.2)))
   )
-  (gr_text "REV B" (at 44.35 33.06) (layer "F.SilkS")
+  (gr_text "REV B" (at 44.36 33.45) (layer "F.SilkS")
     (effects (font (size 1.5 1.5) (thickness 0.2)))
   )
