File: schematics/master_board/master_board.kicad_sch (KiCad schematic)
At the start: 49 parts, among them J1 USB_C_Receptacle_USB2.0, J2 Conn_01x04_Male, J3 Conn_01x04_Female, SW1 SW_Push, SW2 SW_Push, SW3 SW_Push, U1 NCP1117-3.3_SOT223, U2 RP2040, U3 W25Q16JVSSIQ, Y1 ABLS-12.000MHZ-B4-T

Commit message: initial master board rev b
Parts:
- removed J2: Conn_01x04_Male, Connector_PinHeader_2.54mm:PinHeader_1x04_P2.54mm_Vertical, symbol Connector:Conn_01x04_Male
- removed J3: Conn_01x04_Female, Connector_PinHeader_2.54mm:PinHeader_1x04_P2.54mm_Vertical, symbol Connector:Conn_01x04_Female
- removed R6: 49R9, Resistor_SMD:R_0402_1005Metric, symbol Device:R
- added J1: Conn_01x03_MountingPin, Connector_JST:JST_SH_BM03B-SRSS-TB_1x03-1MP_P1.00mm_Vertical, symbol Connector_Generic_MountingPin:Conn_01x03_MountingPin
- added J3: Conn_01x04_Male, Connector_PinHeader_2.54mm:PinHeader_1x04_P2.54mm_Vertical, symbol Connector:Conn_01x04_Male
- added TP1, TP2, TP3: TestPoint, TestPoint:TestPoint_Pad_2.5x2.5mm, symbol Connector:TestPoint
- R11: renamed from R12; value 1k -> 10k
- R14: renamed from R15; value DNF -> 10k
- R15: renamed from R16; value 1k -> 49R9
- R16: renamed from R17; value 1k -> 49R9
- R8: renamed from R9; value 1k -> 10k
- renumbered J1 to J2, R11 to R10, R13 to R12, R14 to R13, R7 to R6, R8 to R7, R10 to R9
Connections:
- net BOOTSEL_N: now also TP3.1
- net CONN_HAP_L: now also J3.4 (Pin_4)
- net CONN_HAP_R: now also J3.1 (Pin_1)
- net CONN_SWCLK: now also J1.1 (Pin_1)
- net CONN_SWDIO: now also J1.3 (Pin_3)
- net GND: now also J1.2 (Pin_2), J3.2 (Pin_2), J3.3 (Pin_3)
- net RESCAN_N: now also TP1.1
- net RUN_N: now also TP2.1
- net GPIO0: no longer names the net of U2.2 (GPIO0)
- net GPIO1: no longer names the net of U2.3 (GPIO1)
- net GPIO13: no longer names the net of U2.16 (GPIO13)
- net GPIO14: no longer names the net of U2.17 (GPIO14)
- net GPIO15: no longer names the net of U2.18 (GPIO15)
- net GPIO20: no longer names the net of U2.31 (GPIO20)
- net GPIO21: no longer names the net of U2.32 (GPIO21)
- net GPIO22: no longer names the net of U2.34 (GPIO22)
- net GPIO23: no longer names the net of U2.35 (GPIO23)
- net GPIO24: no longer names the net of U2.36 (GPIO24)
- net GPIO25: no longer names the net of U2.37 (GPIO25)
- net GPIO26_ADC0: no longer names the net of U2.38 (GPIO26_ADC0)
- net GPIO27_ADC1: no longer names the net of U2.39 (GPIO27_ADC1)
- net GPIO28_ADC2: no longer names the net of U2.40 (GPIO28_ADC2)
- net GPIO29_ADC3: no longer names the net of U2.41 (GPIO29_ADC3)
Other:
- moved on the sheet: R5

Commit message: add gerbers
Changed lines of the file:
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@@
+    (stroke (width 0) (type default) (color 0 0 0 0))
+  )
+  (wire (pts (xy 237.49 101.6) (xy 237.49 100.33))
     (stroke (width 0) (type default) (color 0 0 0 0))
   )
@@
     (pin "2")
   )
-  (symbol (lib_id "power:GND") (at 237.49 100.33 0) (unit 1)
-    (in_bom yes) (on_board yes) (fields_autoplaced)
-    (property "Reference" "#PWR025" (id 0) (at 237.49 106.68 0)
-      (effects (font (size 1.27 1.27)) hide)
-    )
-    (property "Value" "GND" (id 1) (at 237.49 105.41 0)
-      (effects (font (size 1.27 1.27)) hide)
-    )
-    (property "Footprint" "" (id 2) (at 237.49 100.33 0)
-      (effects (font (size 1.27 1.27)) hide)
-    )
-    (property "Datasheet" "" (id 3) (at 237.49 100.33 0)
-      (effects (font (size 1.27 1.27)) hide)
-    )
+  (symbol (lib_id "power:GND") (at 237.49 101.6 0) (unit 1)
+    (in_bom yes) (on_board yes) (fields_autoplaced)
+    (property "Reference" "#PWR025" (id 0) (at 237.49 107.95 0)
+      (effects (font (size 1.27 1.27)) hide)
+    )
+    (property "Value" "GND" (id 1) (at 237.49 106.68 0)
+      (effects (font (size 1.27 1.27)) hide)
+    )
+    (property "Footprint" "" (id 2) (at 237.49 101.6 0)
+      (effects (font (size 1.27 1.27)) hide)
+    )
+    (property "Datasheet" "" (id 3) (at 237.49 101.6 0)
+      (effects (font (size 1.27 1.27)) hide)
+    )
